File: cap_multiplier_tile/V0.1.X/cap_multiplier_tile.kicad_sch (KiCad schematic)
At the start: 9 parts, among them J1 cap_multiplier_board

Commit message: adding action, removing library dependancy
Parts:
- TP1, TP2, TP3, TP4, TP5, TP6, TP7, TP8: footprint EOI:TestPoint_Pad_D1.0mm -> Library:TestPoint_Pad_D1.0mm
Changed lines of the file:
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@@
 			)
 		)
-		(property "Footprint" "EOI:TestPoint_Pad_D1.0mm"
+		(property "Footprint" "Library:TestPoint_Pad_D1.0mm"
 			(at 137.16 125.73 0)
 			(effects
@@
 		)
 		(property "Manufacturer" ""
+			(at 137.16 120.65 0)
+			(effects
+				(font
+					(size 1.27 1.27)
+				)
+				(hide yes)
+			)
+		)
+		(property "Manufacturer Part Number" ""
 			(at 137.16 120.65 0)
 			(effects
@@
 			)
 		)
-		(property "Footprint" "EOI:TestPoint_Pad_D1.0mm"
+		(property "Footprint" "Library:TestPoint_Pad_D1.0mm"
 			(at 143.51 110.49 0)
 			(effects
@@
 		)
 		(property "Manufacturer" ""
+			(at 143.51 115.57 0)
+			(effects
+				(font
+					(size 1.27 1.27)
+				)
+				(hide yes)
+			)
+		)
+		(property "Manufacturer Part Number" ""
 			(at 143.51 115.57 0)
 			(effects
@@
 			)
 		)
-		(property "Footprint" "EOI:TestPoint_Pad_D1.0mm"
+		(property "Footprint" "Library:TestPoint_Pad_D1.0mm"
 			(at 151.13 113.03 0)
 			(effects
@@
 		)
 		(property "Manufacturer" ""
+			(at 151.13 118.11 0)
+			(effects
+				(font
+					(size 1.27 1.27)
+				)
+				(hide yes)
+			)
+		)
+		(property "Manufacturer Part Number" ""
 			(at 151.13 118.11 0)
 			(effects
@@
 			)
 		)
-		(property "Footprint" "EOI:TestPoint_Pad_D1.0mm"
+		(property "Footprint" "Library:TestPoint_Pad_D1.0mm"
 			(at 151.13 107.95 0)
 			(effects
@@
 		)
 		(property "Manufacturer" ""
+			(at 151.13 113.03 0)
+			(effects
+				(font
+					(size 1.27 1.27)
+				)
+				(hide yes)
+			)
+		)
+		(property "Manufacturer Part Number" ""
 			(at 151.13 113.03 0)
 			(effects
@@
 		(property "Description" "Generic connector, double row, 02x04, counter clockwise pin numbering scheme (similar to DIP package numbering), script generated (kicad-library-utils/schlib/autogen/connector/)"
 			(at 158.75 115.57 0)
+			(effects
+				(font
+					(size 1.27 1.27)
+				)
+				(hide yes)
+			)
+		)
+		(property "Manufacturer Part Number" ""
+			(at 160.02 115.57 0)
 			(effects
 				(font
@@
 			)
 		)
-		(property "Footprint" "EOI:TestPoint_Pad_D1.0mm"
+		(property "Footprint" "Library:TestPoint_Pad_D1.0mm"
 			(at 176.53 110.49 0)
 			(effects
@@
 		)
 		(property "Manufacturer" ""
+			(at 176.53 115.57 0)
+			(effects
+				(font
+					(size 1.27 1.27)
+				)
+				(hide yes)
+			)
+		)
+		(property "Manufacturer Part Number" ""
 			(at 176.53 115.57 0)
 			(effects
@@
 			)
 		)
-		(property "Footprint" "EOI:TestPoint_Pad_D1.0mm"
+		(property "Footprint" "Library:TestPoint_Pad_D1.0mm"
 			(at 168.91 113.03 0)
 			(effects
@@
 		)
 		(property "Manufacturer" ""
+			(at 168.91 118.11 0)
+			(effects
+				(font
+					(size 1.27 1.27)
+				)
+				(hide yes)
+			)
+		)
+		(property "Manufacturer Part Number" ""
 			(at 168.91 118.11 0)
 			(effects
@@
 			)
 		)
-		(property "Footprint" "EOI:TestPoint_Pad_D1.0mm"
+		(property "Footprint" "Library:TestPoint_Pad_D1.0mm"
 			(at 168.91 107.95 0)
 			(effects
@@
 		)
 		(property "Manufacturer" ""
+			(at 168.91 113.03 0)
+			(effects
+				(font
+					(size 1.27 1.27)
+				)
+				(hide yes)
+			)
+		)
+		(property "Manufacturer Part Number" ""
 			(at 168.91 113.03 0)
 			(effects
@@
 			)
 		)
-		(property "Footprint" "EOI:TestPoint_Pad_D1.0mm"
+		(property "Footprint" "Library:TestPoint_Pad_D1.0mm"
 			(at 182.88 125.73 0)
 			(effects
@@
 			(at 182.88 120.65 0)
 			(effects
+				(font
+					(size 1.27 1.27)
+				)
+				(hide yes)
+			)
+		)
+		(property "Manufacturer Part Number" ""
+			(at 182.88 120.65 0)
+			(effects
